File: stm32f407_tft_2.4inch_hat/stm32f407_tft_2.4inch_hat.kicad_pcb (KiCad board)
At the start: 2 copper layers, 62.7 x 90.2 mm, 6 parts, among them P1 STM32F407-DISC P1, P2 STM32F407-DISC P2, U1 TFT SPI 240x320

Commit message: PCB wired
Parts:
- moved UART1 33.3 mm to (161.9, 52.6)
- moved I2C-Sensor1 15.7 mm to (128.7, 52.6)
- moved I2C-RealTime1 15.5 mm to (145.2, 52.6)
- renumbered U1 to LCD_Panel1
Connections:
- LCD_Panel1 pad 10: /LCD_T_CLK -> /LCD_SD_CLK
- LCD_Panel1 pad 12: /LCD_T_MOSI -> /LCD_SD_MOSI
- LCD_Panel1 pad 13: /LCD_T_MISO -> /LCD_SD_MISO
- P1 pad 11: /LCD_T_IRQ -> /PC13
- P1 pad 13: /LCD_T_CS -> /LCD_T_IRQ
- P1 pad 15: /PE1 -> /LCD_T_CS
- P1 pad 17: /LCD_CS -> /PE1
- P1 pad 19: /VDD -> /LCD_CS
- P1 pad 21: /PB7 -> unconnected-(P1-BOOT0-Pad21)
- P1 pad 23: /PB5 -> /PB7
- P1 pad 25: /PB3 -> /PB5
- P1 pad 27: /PD6 -> /PB3
- P1 pad 29: /PD4 -> /PD6
- P1 pad 31: /PD2 -> /PD4
- P1 pad 33: /PD0 -> /PD2
- P1 pad 35: /LCD_SD_MISO -> /PD0
- P1 pad 37: /PA15 -> /LCD_SD_MISO
- P1 pad 39: /PA13 -> /PA15
- P1 pad 41: /PA9 -> /PA13
- P1 pad 43: /PC9 -> /PA9
- P1 pad 45: /PC7 -> /PC9
- P1 pad 47: /GND -> /PC7
Routing:
- net /LCD_SD_MOSI: track 0.00 -> 129.8 mm, vias 0 -> 4
- net /LCD_SD_MISO: track 0.00 -> 119.3 mm, vias 0 -> 4
- net /I2C2_SCL: track 0.00 -> 116.6 mm, vias 0 -> 2
- net /I2C2_SDA: track 0.00 -> 113.9 mm, vias 0 -> 2
- net /LCD_SD_CLK: track 0.00 -> 104.3 mm, vias 0 -> 4
- net /LCD_T_IRQ: track 0.00 -> 91.3 mm, vias 0 -> 4
- net /5V: track 0.00 -> 89.3 mm
- net /LCD_T_CS: track 0.00 -> 81.9 mm, vias 0 -> 4
- net /3V: track 0.00 -> 70.8 mm, vias 0 -> 2
- net /LCD_SD_CS: track 0.00 -> 68.9 mm, vias 0 -> 1
- net /LCD_MISO: track 0.08 -> 68.7 mm
- net /LCD_CS: track 0.00 -> 54.8 mm, vias 0 -> 1
- net /DBG_UART2_TX: track 0.15 -> 49.2 mm
- net /LCD_SCK: track 0.00 -> 43.6 mm, vias 0 -> 5
- net /LCD_MOSI: track 0.13 -> 42.5 mm, vias 0 -> 1
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- added copper zone on B.Cu, net /GND

Commit message: Final state and export gerber
Connections:
- P2 pad 13: /DBG_UART2_RX -> /DBG_UART2_TX
- P2 pad 14: /DBG_UART2_TX -> /DBG_UART2_RX
Routing:
- net /DBG_UART2_RX: track 41.7 -> 46.2 mm
- net /DBG_UART2_TX: track 49.2 -> 46.7 mm
- net /LCD_T_CS: track 81.9 -> 81.4 mm
- net /LCD_SCK: vias 5 -> 4
Other:
- board text added: "3.3V"
- board text added: "RX"
- board text added: "SCL"
- board text added: "SDA"
- board text added: "TX"
- board text removed: "PC13"
